File: Michal/SmartTrashCan/SmartTrashCan.kicad_sch (KiCad schematic)
At the start: 23 parts, among them J1 USB_C_Receptacle_USB2.0_16P, J2 USB_C_Receptacle_USB2.0_16P, U1 ESP32-C6-WROOM-1, U2 AZ1117-3.3, U3 CP2102N-Axx-xQFN20

Commit message: Summary
All around ESP32
Parts:
- added C10, C7, C8, C9: 1uF, symbol Device:C
- added C5, C6: 10uF, symbol Device:C
- added R3: 22.1K, symbol Device:R
- added R6: 47.5k, symbol Device:R
- added R7: 1K, symbol Device:R
- added R8, R9: 10K, symbol Device:R
- added SW1, SW2: SW_Push, symbol Switch:SW_Push
Connections:
- net +3V3: now also U1.2 (3V3), U3.6 (VDD), U3.7 (VREGIN), C6.1, C7.2, R7.1, R9.1
- net +5V: now also C1.1, U2.3 (VI)
- net ESP32_D+: now also U1.14 (GPIO13/USB_D+)
- net ESP32_D-: now also U1.13 (GPIO12/USB_D-)
- net GND: now also U1.1 (GND), U1.28 (GND), U1.29 (GND), U3.12 (GND), U3.21 (GND), U3.3 (GND), C10.1, C5.2, C6.2, C7.1, C8.2, C9.1, R6.1, R8.2, SW1.2, SW2.2
- net VBUSA: now also R3.1
- net at U3.11 (~{SUSPEND}): now also R8.1
- net USB_UART_RX: now reaches U3.17 (RXD)
- net USB_UART_RX: now also U1.25 (U0TXD/GPIO16)
- net USB_UART_TX: now reaches U3.18 (TXD)
- net USB_UART_TX: now also U1.24 (U0RXD/GPIO17)
- net at U3.8 (VBUS): now also C5.1, R3.2, R6.2
- net at U3.9 (~{RST}): now also R7.2
- net BOOT: now reaches U1.15 (GPIO9)
- net BOOT: now also C10.2, SW2.1
- net RESET: now reaches U1.3 (EN/CHIP_PU)
- net RESET: now also C8.1, C9.2, R9.2, SW1.1
- no-connect marks 4 -> 12
Other:
- note added: "LDO"
- moved on the sheet: C1, C2, U2

Commit message: Update SmartTrashCan.kicad_sch
Other:
- note added: "ESP32-C6"
- moved on the sheet: C10, C7, C8, C9, R9, SW1, SW2, U1
