File: GamingControler/_autosave-GamingControler.kicad_pcb (KiCad board)
At the start: 2 copper layers, 40 x 55 mm, 36 parts, among them J1 USB_C_Receptacle_USB2.0_16P, J2 USB_C_Receptacle_USB2.0_16P, SW1 SW_Push, SW2 SW_Push, U1 ESP32-C6-WROOM-1, U2 AZ1117-3.3, U3 CP2102N-Axx-xQFN20

Commit message: Final board
Parts:
- removed JP1, JP2: SolderJumper_2_Open, Jumper:SolderJumper-2_P1.3mm_Open_TrianglePad1.0x1.5mm
- added C11: 10nF, Capacitor_SMD:C_0805_2012Metric, F.Cu at (40.0, 49.5)
- added C12: 10nF, Capacitor_SMD:C_0805_2012Metric, F.Cu at (40.0, 62.5)
- added C13: 50pF, Capacitor_SMD:C_0805_2012Metric, F.Cu at (36.5, 49.5)
- added C14: 50pF, Capacitor_SMD:C_0805_2012Metric, F.Cu at (36.5, 62.5)
- added C15: 10nF, Capacitor_SMD:C_0805_2012Metric, F.Cu at (39.5, 75.5)
- added C16: 50pF, Capacitor_SMD:C_0805_2012Metric, F.Cu at (36.5, 75.5)
- added C17: 10nF, Capacitor_SMD:C_0805_2012Metric, F.Cu at (40.0, 88.5)
- added C18: 50pF, Capacitor_SMD:C_0805_2012Metric, F.Cu at (36.5, 88.5)
- added E1: ~, LED_SMD:Electrode_10x10mm, F.Cu at (28.7, 43.1)
- added E2: ~, LED_SMD:Electrode_10x10mm, F.Cu at (28.7, 56.1)
- added E3: ~, LED_SMD:Electrode_10x10mm, F.Cu at (28.7, 69.1)
- added E4: ~, LED_SMD:Electrode_10x10mm, F.Cu at (28.7, 82.1)
- added J3: Conn_01x05_Pin, Connector_PinHeader_2.54mm:PinHeader_1x05_P2.54mm_Vertical, F.Cu at (25.9, 96.0)
- added J4: Conn_01x05_Pin, Connector_PinHeader_2.54mm:PinHeader_1x05_P2.54mm_Vertical, F.Cu at (25.9, 39.0)
- added U4: TTP223-BA6, Package_TO_SOT_SMD:TSOT-23-6_HandSoldering, F.Cu at (38.5, 45.5)
- added U5: TTP223-BA6, Package_TO_SOT_SMD:TSOT-23-6_HandSoldering, F.Cu at (38.5, 58.5)
- added U6: TTP223-BA6, Package_TO_SOT_SMD:TSOT-23-6_HandSoldering, F.Cu at (38.5, 71.5)
- added U7: TTP223-BA6, Package_TO_SOT_SMD:TSOT-23-6_HandSoldering, F.Cu at (38.5, 84.5)
Connections:
- J1 pad S1: Net-(J1-SHIELD) -> GND
- J2 pad S1: Net-(J2-SHIELD) -> GND
- U1 pad 23: unconnected-(U1-GPIO15-Pad23) -> OUTPUT
Routing:
- net +3V3: track 6.06 -> 180.6 mm, vias 0 -> 5
- net V_X_L: track 0.00 -> 49.6 mm, vias 0 -> 1
- net V_Y_L: track 0.00 -> 48.3 mm, vias 0 -> 1
- net Push_L: track 0.00 -> 47.1 mm, vias 0 -> 1
- net V_X_R: track 0.00 -> 39.7 mm, vias 0 -> 1
- net V_Y_R: track 0.00 -> 38.5 mm, vias 0 -> 1
- net Push_R: track 0.00 -> 37.1 mm, vias 0 -> 1
- net OUTPUT4: track 0.00 -> 35.2 mm, vias 0 -> 2
- net OUTPUT1: track 0.00 -> 34.8 mm, vias 0 -> 2
- net OUTPUT3: track 0.00 -> 22.4 mm, vias 0 -> 2
- net OUTPUT2: track 0.00 -> 21.6 mm, vias 0 -> 2
- net BOOT: track 28.1 -> 36.4 mm, vias 0 -> 2
- net RESET: track 10.4 -> 18.3 mm
- net ANTENNA4: track 0.00 -> 4.70 mm
- net ANTENNA3: track 0.00 -> 4.70 mm
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- added copper zone on B.Cu, net GND
- added copper zone on F.Cu, net GND
Other:
- board size 40 x 55 mm -> 53 x 63 mm
